File: nixie2.sch (EAGLE design)
At the start: 36 parts, among them IC1 74141N, IC2 MEGA16-P, IC3 74141N, IC4 74141N, IC5 74141N, IC6 74141N, IC7 74141N, IC8 7805T, Q1 IRF840, X1 332-02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

Commit message: Schematic printout
Other:
- note added: "Copyright (c) 2014 Chris Fallin <cfallin@c1f.net>"
- note added: "NIXIE CLOCK"
Changed lines of the file:
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@@
 <sheet>
 <plain>
+<text x="27.94" y="91.44" size="7.62" layer="91">NIXIE CLOCK</text>
+<text x="-2.54" y="81.28" size="5.08" layer="91">Copyright (c) 2014 Chris Fallin &lt;cfallin@c1f.net&gt;</text>
 </plain>
 <instances>
